File: eagle/FanController.brd (EAGLE design)
At the start: 45 x 20 mm, 14 parts, among them IC102 LDK320AM33R, IC201 STM32F042G6U6

Commit message: - converted to 4 layer board and sent to FAB - coded ADC temperature calculations (timer1) - coded RPM calculations (timer2)
Parts:
- removed SV301: n/a, pinhead:1X04
- added C407, C507, C607: 1u, rcl:C0805
- added DEBUG200: LSP10, solpad:LSP10
- added J301: 47053-1000, 47053-1000:470531000
- added LED801: APHBM2012SURKZGKC, APHBM2012LSURKZGKC:SMD
- added R301: 10k, rcl:R0805
- added R802: 68R, rcl:R0805
- moved C207 1.00 mm to (27.0, 9.00), turned to 0 degrees
- renumbered POWER to JP1, SWD101 to SWD1
Connections:
- new net LED1:R_A: LED801.1, R802.2
- new net LED_GREEN: IC201.7_PA1, LED801.3
- new net LED_RED: IC201.6_PA0, LED801.2
- new net STM32:DEBUG_OUT: DEBUG200.MP, IC201.23_PA15
- net 3V3: now also LED801.4, R301.2, R802.1
- net FAN_PWM: now also J301.4; no longer SV301.3
- net FAN_TACHO: now also J301.3, R301.1; no longer SV301.2
- net GND: now also C407.1, C507.1, C607.1, J301.1; no longer SV301.1
- net TEMP1: now also C407.2
- net TEMP2: now also C507.2
- net TEMP3: now also C607.2
- net VDD: now also J301.2; no longer SV301.4
Routing:
- net 3V3: track 72.1 -> 17.1 mm, vias 4 -> 6
- net LED_RED: track 0.00 -> 10.4 mm, vias 0 -> 2
- net FAN_TACHO: track 24.5 -> 33.0 mm, vias 0 -> 2
- net LED_GREEN: track 0.00 -> 8.00 mm, vias 0 -> 2
- net TEMP3: track 18.3 -> 22.7 mm, vias 0 -> 1
- net TEMP1: track 7.58 -> 12.0 mm, vias 0 -> 1
- net STM32:DEBUG_OUT: track 0.00 -> 4.08 mm
- net TEMP2: track 9.26 -> 13.2 mm, vias 0 -> 1
- net VDD: track 55.0 -> 58.8 mm, vias 0 -> 1
- net SYS_SWCLK: track 12.1 -> 9.28 mm, vias 1 -> 2
- net LED1:R_A: track 0.00 -> 1.54 mm
- net FAN_PWM: track 24.5 -> 25.7 mm, vias 0 -> 1
- net GND: vias 35 -> 32
- added copper zone on layer 2, net 3V3
- added copper zone on layer 15, net GND
Other:
- board text added: "debug_out"
