File: eagle/FanController.sch (EAGLE design)
At the start: 2 parts

Commit message: rev.2: PWM fan a PWM fan shall be connected to the controller
- initialized all unused pins as analog
- removed FET for transistor control
- added noctua PWM specification white paper
- rev.2 board marking on tstop
- replaced connectors with pin headers
Parts:
- POWER: value 22-23-2021 -> n/a; device con-molex:22-23-2021 -> pinhead:PINHD-1X2
Connections:
- net GND: now also POWER.1; no longer POWER-1.S
- net VDD: now also POWER.2; no longer POWER-2.S

Commit message: - converted to 4 layer board and sent to FAB - coded ADC temperature calculations (timer1) - coded RPM calculations (timer2)
Parts:
- removed POWER: n/a, pinhead:PINHD-1X2
- removed SWD101: TC2030-NL, tag-connect:TC2030
- added JP1: n/a, pinhead:PINHD-1X2
- added SWD1: TC2030-NL, tag-connect:TC2030
Connections:
- net 3V3: now also SWD1.1_T_VCC; no longer SWD101.1_T_VCC
- net GND: now also JP1.1, SWD1.5_GND; no longer POWER.1, SWD101.5_GND
- net SYS_NRST: now also SWD1.3_T-NRST; no longer SWD101.3_T-NRST
- net SYS_SWCLK: now also SWD1.4_T-SWCLK; no longer SWD101.4_T-SWCLK
- net SYS_SWDIO: now also SWD1.2_T-SWDIO; no longer SWD101.2_T-SWDIO
- net VDD: now also JP1.2; no longer POWER.2
Other:
- note added: "10k, 0.25W, 0805"
- note added: "R"
- note added: "connect via low pass filter fcutoff = 15.9 Hz R=10k TH, C=1uF TH"
