File: eagle/FanController.sch (EAGLE design)
At the start: 2 parts

Commit message: - coded ADC temperature calculations (timer1) - coded RPM calculations (timer2)
Parts:
- removed POWER: n/a, pinhead:PINHD-1X2
- added JP101: n/a, pinhead:PINHD-1X2
Connections:
- net GND: now also JP101.1; no longer POWER.1
- net VDD: now also JP101.2; no longer POWER.2
Other:
- note added: "connect via low pass filter fcutoff = 15.9 Hz R=10k TH, C=1uF TH"
